File: compact_sqm/compact_sqm.kicad_sch (KiCad schematic)
At the start: 6 parts, among them J1 USB4135-GF-A, U1 TSL25911FN, U2 MCP73831-2-OT, U3 ESP-12F, U4 CH340C

Commit message: schematic edits
Parts:
- removed J1: USB4135-GF-A, Connector_USB:USB_C_Receptacle_GCT_USB4135-GF-A_6P_TopMnt_Horizontal, symbol Connector:USB_C_Receptacle_PowerOnly_6P
- added C1, C2: 10uF, Capacitor_SMD:C_0603_1608Metric, symbol Device:C_Small
- added C3: 0.1uF, Capacitor_SMD:C_0603_1608Metric, symbol Device:C_Small
- added J1: USB_C_Receptacle_USB2.0_16P, Connector_USB:USB_C_Receptacle_GCT_USB4110, symbol Connector:USB_C_Receptacle_USB2.0_16P
- added Q1, Q2: MMBT3904, Package_TO_SOT_SMD:SOT-23, symbol Transistor_BJT:MMBT3904
- added R1, R2: 5.1K, Resistor_SMD:R_0603_1608Metric, symbol Device:R_US
- added R3, R4: 499, Resistor_SMD:R_0603_1608Metric, symbol Device:R_US
- added R5, R6: 12K, Resistor_SMD:R_0603_1608Metric, symbol Device:R_US
- added U5: TLV70233DBVR, Package_TO_SOT_SMD:SOT-23-5, symbol Regulator_Linear:TLV70233_SOT23-5
Connections:
- net GND: now reaches U2.2 (V_{SS})
- net GND: now also BT1.2 (-), U1.3 (GND), U4.1 (GND), C1.2, C2.2, C3.2, J1.A1 (GND), J1.A12 (GND), J1.B1 (GND), J1.B12 (GND), J1.S1 (SHIELD), R1.2, R2.2
- net VBAT: now reaches U2.3 (V_{BAT})
- net VBAT: now also BT1.1 (+)
- net VBUS: now reaches U2.4 (V_{DD})
- net VBUS: now also U4.16 (VCC), C1.1
- net RXD: now reaches U3.21 (GPIO3/RXD)
- net RXD: now also R3.2
- net TXD: now reaches U3.22 (GPIO1/TXD)
- net TXD: now also R4.2
- net at U3.8 (VCC): now also C2.1
- net at U1.5 (VDD): now also C3.1
- net at U4.2 (TXD): now also R3.1
- net at U4.3 (RXD): now also R4.1
- net at U4.5 (UD+): now also J1.A6 (D+), J1.B6 (D+)
- net at U4.6 (UD-): now also J1.A7 (D-), J1.B7 (D-)
- new net: J1.A4 (VBUS), J1.A9 (VBUS), J1.B4 (VBUS), J1.B9 (VBUS)
- new net: J1.A5 (CC1), R1.1
- new net: J1.B5 (CC2), R2.1
- new net: Q2.1 (B), R5.1, R6.2
- new net: Q1.1 (B), R5.2, R6.1
- new net +3.3V: U5.5 (OUT)
Other:
- moved on the sheet: U1, U3, U4

Commit message: finished schematic
Parts:
- added C4: 10uF, Capacitor_SMD:C_0603_1608Metric, symbol Device:C_Small
- added C5, C6, C7, C8: 0.1uF, Capacitor_SMD:C_0603_1608Metric, symbol Device:C_Small
- added D1: LED, LED_SMD:LED_0603_1608Metric_Pad1.05x0.95mm_HandSolder, symbol Device:LED
- added R10, R11, R12, R13, R7, R8, R9: 12K, Resistor_SMD:R_0603_1608Metric, symbol Device:R_US
- added SW1: SW_SPDT, Button_Switch_SMD:SW_SPDT_PCM12, symbol Switch:SW_SPDT
- BT1: footprint (none) -> Connector_PinHeader_2.54mm:PinHeader_2x01_P2.54mm_Vertical
Connections:
- net +3.3V: now also C2.1, C3.1, U1.5 (VDD), U3.8 (VCC), C5.1, R10.2, R11.2, R13.1, R9.2
- net GND: now also U3.15 (GND), U5.2 (GND), C4.2, C5.2, C6.2, C7.2, C8.2, R12.2, R7.1
- net VBAT: now also U5.1 (IN), U5.3 (EN), C4.1, C6.1, SW1.2 (B); no longer BT1.1 (+)
- net VBUS: now also J1.A4 (VBUS), J1.A9 (VBUS), J1.B4 (VBUS), J1.B9 (VBUS), C7.1, D1.2 (A)
- net RST: now reaches U3.1 (~{RST})
- net RST: now also Q1.3 (C)
- net at U3.16 (GPIO15): now also R12.1
- net SDA: now reaches U3.17 (GPIO2)
- net SDA: now also U1.6 (SDA), R9.1
- net BOOT: now reaches U3.18 (GPIO0)
- net BOOT: now also Q2.3 (C)
- net INT: now reaches U3.19 (GPIO4)
- net INT: now also U1.2 (INT), R11.1
- net at U3.3 (EN): now also R13.2
- net SCL: now reaches U3.5 (GPIO14)
- net SCL: now also U1.1 (SCL), R10.1
- net at U2.1 (STAT): now also R8.2
- net at U2.5 (PROG): now also R7.2
- net at U4.13 (~{DTR}): now also Q2.2 (E), R5.1
- net at U4.14 (~{RTS}): now also Q1.2 (E), R6.1
- net at U4.4 (V3): now also C8.1
- net at Q2.1 (B), R6.2: no longer R5.1
- net at Q1.1 (B), R5.2: no longer R6.1
- new net: D1.1 (K), R8.1
- new net: BT1.1 (+), SW1.1 (A)
- no-connect marks 0 -> 7
Other:
- moved on the sheet: BT1, C1, U2

Commit message: layout updates
Parts:
- added H1, H2, H3, H4: M2, MountingHole:MountingHole_2.2mm_M2, symbol Mechanical:MountingHole
Connections:
- no-connect marks 7 -> 18
