File: compact_sqm/compact_sqm.kicad_pcb (KiCad board)
At the start: 2 copper layers, 32 parts, among them J1 USB_C_Receptacle_USB2.0_16P, Q1 MMBT3904, Q2 MMBT3904, SW1 SW_SPDT, U1 TSL25911FN, U2 MCP73831-2-OT, U3 ESP-12F, U4 CH340C, U5 TLV70233DBVR

Commit message: layout updates
Parts:
- added H1: M2, MountingHole:MountingHole_2.2mm_M2, F.Cu at (129.3, 78.5)
- added H2: M2, MountingHole:MountingHole_2.2mm_M2, F.Cu at (150.1, 78.5)
- added H3: M2, MountingHole:MountingHole_2.2mm_M2, F.Cu at (150.1, 124.7)
- added H4: M2, MountingHole:MountingHole_2.2mm_M2, F.Cu at (129.3, 124.7)
- moved R1 66.1 mm to (139.4, 117.6)
- moved R2 63.8 mm to (142.5, 117.6)
- moved C1 63.2 mm to (150.7, 112.2)
- moved R7 59.6 mm to (150.7, 110.4), turned to 180 degrees
- moved R8 57.4 mm to (143.9, 111.3), turned to 90 degrees
- moved C4 57.2 mm to (145.8, 114.8), turned to -90 degrees
- moved C2 50.2 mm to (129.5, 104.1), turned to -90 degrees
- moved SW1 48.0 mm to (150.4, 117.6)
- moved BT1 47.9 mm to (130.0, 119.9), turned to 90 degrees
- moved C5 47.2 mm to (146.1, 106.9)
- moved C8 46.6 mm to (136.1, 117.6), turned to 180 degrees
- moved C6 46.2 mm to (146.1, 108.5)
- moved J1 46.2 mm to (139.7, 123.3)
- moved R5 46.1 mm to (138.2, 107.7), turned to 90 degrees
- moved R6 43.6 mm to (136.4, 107.7), turned to 90 degrees
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Routing:
- net GND: track 0.00 -> 28.1 mm
- net Net-(BT1-+): track 0.00 -> 27.8 mm
Other:
- board outline added: 25.4 x 50.8 mm

Commit message: finished layout
Parts:
- moved C5 5.12 mm to (151.1, 106.0), turned to 90 degrees
- moved U5 2.06 mm to (148.1, 107.7)
- moved C6 1.47 mm to (144.7, 107.8), turned to 90 degrees
- moved Q1 0.13 mm to (129.9, 110.0)
- moved Q2 0.13 mm to (129.9, 113.5)
Routing:
- net GND: track 28.1 -> 170.4 mm, vias 0 -> 10
- net +3.3V: track 0.00 -> 68.5 mm
- net VBUS: track 0.00 -> 43.4 mm, vias 0 -> 2
- net Net-(U4-RXD): track 0.00 -> 36.4 mm, vias 0 -> 2
- net Net-(U4-TXD): track 0.00 -> 34.6 mm, vias 0 -> 2
- net SDA: track 0.00 -> 32.2 mm, vias 0 -> 2
- net INT: track 0.00 -> 30.3 mm, vias 0 -> 2
- net SCL: track 0.00 -> 28.5 mm, vias 0 -> 2
- net BOOT: track 0.00 -> 27.6 mm, vias 0 -> 2
- net RST: track 0.00 -> 24.5 mm, vias 0 -> 2
- net VBAT: track 0.00 -> 16.6 mm
- net Net-(Q2-B): track 0.00 -> 13.1 mm
- net Net-(Q2-E): track 0.00 -> 12.6 mm
- net Net-(Q1-E): track 0.00 -> 11.2 mm
- net Net-(Q1-B): track 0.00 -> 10.8 mm
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Other:
- outline, holes or cut-outs redrawn
- board text added: "+"
- board text added: "-"
- board text added: "Compact SQM"
- board text added: "Compact Sky Quality Meter"
- board text added: "Jannett W"
